File: KiCad/CherryZXKeyboard.kicad_pcb (KiCad board)
At the start: 2 copper layers, 290 x 120 mm, 104 parts, among them J1 Conn_01x05_Female, J2 Conn_01x08_Female, SW1 1, SW10 E, SW11 D, SW12 X, SW13 4, SW14 R, SW15 F, SW16 C, SW17 5, SW18 T, SW19 G, SW2 Q, SW20 V, SW21 6, SW22 Y, SW23 H, SW24 B, SW25 7, SW26 U, SW27 J, SW28 N, SW29 8, SW3 A, SW30 I, SW31 K, SW32 M, SW33 9, SW34 O, SW35 L, SW36 SYM, SW37 0, SW38 P, SW39 ENT, SW4 CAP, SW40 SPC, SW41 CAP, SW42 ;, SW43 ", SW44 ,, SW45 SYM, SW46 BREAK, SW47 EXTEND, SW48 DOT, SW49 LEFT, SW5 2, SW50 INV VID, SW51 TRUE VID, SW52 CAPS LOCK, SW53 EDIT, SW54 DOWN, SW55 UP, SW56 RIGHT, SW57 GRAPH, SW58 DEL, SW6 W, SW7 S, SW8 Z, SW9 3, U1 4066, U2 4066, U3 4066, U4 4066, U5 4066

Commit message: Change footprints for keys 2U 6.25 U with mechanical stabilizers for PCB mounting
Parts:
- removed the REF** at (321.7, 154.1)
- removed the REF** at (83.7, 174.1)
- removed the REF** at (332.7, 134.1)
- removed the REF** at (63.7, 154.1)
- added REF**: SW_Cherry_MX_1.75u_PCB, Button_Switch_Keyboard:SW_Cherry_MX_1.75u_PCB, F.Cu at (75.6, 154.1)
- added REF**: SW_Cherry_MX_1.75u_PCB, Button_Switch_Keyboard:SW_Cherry_MX_1.75u_PCB, F.Cu at (320.7, 134.2)
- added REF**: SW_Cherry_MX_1.75u_PCB, Button_Switch_Keyboard:SW_Cherry_MX_1.75u_PCB, F.Cu at (309.7, 154.1)
- added REF**: SW_Cherry_MX_1.75u_PCB, Button_Switch_Keyboard:SW_Cherry_MX_1.75u_PCB, F.Cu at (95.6, 174.2)
- SW39, SW4, SW41, SW45: footprint Button_Switch_Keyboard:SW_Cherry_MX_1.00u_PCB -> Button_Switch_Keyboard:SW_Cherry_MX_2.00u_PCB
- SW40: footprint Button_Switch_Keyboard:SW_Cherry_MX_1.00u_PCB -> Button_Switch_Keyboard:SW_Cherry_MX_6.25u_PCB
- moved SW4 9.50 mm to (73.2, 154.1)
- moved SW45 9.50 mm to (93.2, 174.1)
- moved SW39 9.42 mm to (323.1, 134.1)
- moved SW41 9.42 mm to (312.1, 154.1)
Routing:
- net VDD: track 984.8 -> 950.2 mm
- net Net-(D30-A): track 564.5 -> 586.5 mm
- net Net-(D24-A): track 141.9 -> 156.0 mm
- net Net-(D15-K): track 466.1 -> 480.1 mm
- net Net-(D17-K): track 524.6 -> 535.5 mm
- net Net-(D16-K): track 195.1 -> 204.5 mm
- net Net-(D8-A): track 557.1 -> 563.0 mm
- net Net-(D25-A): track 222.6 -> 221.7 mm
- net (no net): vias 6 -> 0
Other:
- board size 290 x 120 mm -> 294 x 127 mm
- board text added: "Cherry ZX Spectrum keyboard 1.1b THT"
- board text removed: "Cherry ZX Spectrum keyboard 1.1 THT"
